File: PCB/MotorController.sch (EAGLE design)
At the start: 68 parts, among them IC1 OPA333D, U1 MIC5235-3.3, U3 SAM3S4/2/1A_48PIN_LQFP, X1 12MHz, X2 08-JST-B8B-XH-A

Commit message: Added 12v power supply, removed CPU in favor of Flutter (for quick development), added headers... many other changes. This commit represents version 0.1 of the hardware.
Parts:
- removed C2, C3: 4.7uF 35v 490-7208-1-ND, Taylor:CAPACITOR0805
- removed C32, C33, C34, C35, C36, C37, C38, C41: 0.1uF, Taylor:CAPACITOR0402
- removed C39, C40: 2.2uF, Taylor:CAPACITOR0402
- removed C42, C43: 15pF, Taylor:CAPACITOR0402
- removed F1: 500mA, Taylor:PTC0603
- removed JP1: M10", SparkFun:M10"
- removed LED1: WS2812, adafruit:WS2812
- removed R21, R6: 1k, Taylor:RESISTOR0402
- removed R22: 2k, Taylor:RESISTOR0402
- removed R5: 6.49k, Taylor:RESISTOR0402
- removed U$10, U$11, U$12: HIGHCURRENTPAD2, Taylor:HIGHCURRENTPAD2
- removed U$2: MICRO_USB, Taylor:MICRO_USB
- removed U$21: XT60, Taylor:XT60
- removed U$8, U$9: MOSFETSO-8, Taylor:MOSFETSO-8
- removed U3: SAM3S4/2/1A_48PIN_LQFP, Taylor:SAM3S4/2/1A_48PIN_LQFP
- added A, B, C: HIGHCURRENTPAD2, Taylor:HIGHCURRENTPAD2
- added AH, AL, BH, BL, CH, CL: MOSFETSO-8, Taylor:MOSFETSO-8
- added CBOOT: 100nF, AcceleratedDesigns:GRM188R72A104KA35D
- added CIN: 2.2uF, AcceleratedDesigns:C3225X7R2A225K230AB
- added COUT: 4.7uF, AcceleratedDesigns:GRM21BR61E475MA12L
- added D10, D11, D12, D13, D8, D9: MBRA140, SparkFun-DiscreteSemi:DIODE-SCHOTTKY-MBRA140
- added JP13, JP14, JP15, JP16, JP17, JP18: M20, SparkFun:M20
- added L1: 82uH, AcceleratedDesigns:ME3220-823KLB
- added RFBB: 6.04k, AcceleratedDesigns:CRCW04026K04FKED
- added RFBT: 88.7k, AcceleratedDesigns:CRCW040288K7FKED
- added SJ1: SOLDERJUMPERNO, SparkFun-Retired:SOLDERJUMPERNO
- added STANDOFF1, STANDOFF2, STANDOFF3, STANDOFF4: STAND-OFF, SparkFun-Electromechanical:STAND-OFF
- added TP1, TP11, TP12, TP13, TP14, TP15, TP2, TP3, TP4, TP5, TP6, TP7, TP8, TP9: TEST_POINT5015KCT-ND, Taylor:TEST_POINT5015KCT-ND
- added X4: 04-JST-B4B-XH-A, con-jst-xh:04-JST-B4B-XH-A
- added X5: USBPTH, SparkFun:USBPTH
- added X6, X7: 05-JST-B5B-XH-A, con-jst-xh:05-JST-B5B-XH-A
- D2: value (none) -> 770mV; device SparkFun:DIODESOD -> AcceleratedDesigns:DFLS1100-7
- R1: value 27R -> 0R; device Taylor:RESISTOR0402 -> Taylor:RESISTOR0603
- R4: value 27R -> DNS; device Taylor:RESISTOR0402 -> Taylor:RESISTOR0603
- U$4: value MOSFETSO-8 -> (none); device Taylor:MOSFETSO-8 -> Taylor:CAPACITOR0805
- U$5: value MOSFETSO-8 -> 470pF; device Taylor:MOSFETSO-8 -> Taylor:CAPACITOR0603-CAP
- U$6: value MOSFETSO-8 -> KMZ60_MAG_ANGLE_SENSOR; device Taylor:MOSFETSO-8 -> Taylor:KMZ60_MAG_ANGLE_SENSOR
- U$7: value MOSFETSO-8 -> 0.22uF; device Taylor:MOSFETSO-8 -> Taylor:CAPACITOR0805
- U1: value MIC5235-3.3 -> Value; device SparkFun:V_REG_LDOSMD -> AcceleratedDesigns:LMR16006YDDCR
- X1: value 12MHz -> 05-JST-B5B-XH-A; device Taylor:XTAL_ABRACON_4_PINABM8G -> con-jst-xh:05-JST-B5B-XH-A
- X2: value 08-JST-B8B-XH-A -> 04-JST-B4B-XH-A; device con-jst-xh:08-JST-B8B-XH-A -> con-jst-xh:04-JST-B4B-XH-A
- renumbered U$19 to -, U$20 to +
Connections:
- net N$1 renamed AHB
- net N$34 renamed CHB
- removed net +1.8V: C32.1, C33.1, C34.1, C35.1, C39.1, U3.VDDCORE@18, U3.VDDCORE@41, U3.VDDOUT, U3.VDDPLL
- removed net +3V3: IC1.V+, LED1.LEDVDD, LED1.VDD
- removed net 3.3V: C3.2, C36.2, C37.1, C38.2, C40.1, C41.2, U1.OUT, U3.ADVREF, U3.VDDIN, U3.VDDIO@13, U3.VDDIO@33, U3.VDDIO@47
- removed net N$10: D2.A, F1.2
- removed net N$16: JP1.7
- removed net N$17: JP1.6
- removed net N$18: JP1.5
- removed net N$2: D1.A, D3.A, D4.A
- removed net N$20: JP1.4
- removed net N$29: JP1.3
- removed net N$3: JP1.10
- removed net N$30: JP1.2
- removed net N$31: JP1.1
- removed net N$35: C42.2, U3.PB8/XOUT, X1.X2
- removed net N$36: C43.2, U3.PB9/XIN, X1.X1
- removed net N$5: JP1.9
- removed net N$6: JP1.8
- removed net RAW: C2.2, D2.C, R5.2, U1.EN, U1.IN
- removed net S0/UVCCDIV: R21.1, R22.2, U3.CTS0/ADTRG/XOUT32/PA8
- removed net S10/CK: U3.SPCK/PWMH3/WKUP8/PA14
- removed net S11/A5: R5.1, R6.2, U3.PWMH1/AD5/PB1
- removed net S4: U3.TF/TIOA1/PWML3/WKUP14/PIODCEN1/PA15
- removed net S6/IO2: U3.UTXD0/NPCS2/PA10
- removed net S7/CS: U3.URXD0/NPCS1/PWMFI0/WKUP6/PA9
- removed net S8/SI: U3.MOSI/PWMH2/PA13
- removed net S9/SO: U3.MISO/PWMH1/PA12
- removed net UDDC_+: R4.2, U3.PB11/DDP
- removed net UDDC_-: R1.2, U3.PB10/DDM
- new net +12V: COUT.1, D1.A, D3.A, D4.A, JP13.19, JP16.19, JP18.19, L1.2, R4.2, RFBT.1, TP8.P$1, U$3.VDD, X1-1.1
- new net 2: RFBB.1, RFBT.2, U1.FB
- new net 3: CBOOT.1, D2.K, L1.1, U1.SW
- new net 5: CBOOT.2, U1.CB
- new net A5: JP14.12, JP15.12, JP17.12, X1-3.1
- new net D11: JP13.5, JP16.5, JP18.5
- new net GND2: U$6.GND, U$7.1, X6-5.1
- new net N$1: U$3.RFSH, U$5.1
- new net RDEL: R1.2, R4.1, U$3.RDEL
- new net S0/CK: JP14.13, JP15.13, JP17.13
- new net S4/IO2: JP14.17, JP15.17, JP17.17
- new net S6/IO0: JP14.19, JP15.19, JP17.19
- new net S7/B: JP13.2, JP16.2, JP18.2
- new net S8/G: JP13.3, JP16.3, JP18.3
- new net S9/R: JP13.4, JP16.4, JP18.4
- new net VCC: IC1.V+, JP13.18, JP16.18, JP18.18, U$4.1, X1-2.1, X2-3.1, X4-3.1, X7-4.1
- new net VCC2: U$6.TCC_EN, U$6.VCC, U$7.2, X6-2.1
- new net VOUT1: U$6.VOUT1, X6-3.1
- new net VOUT2: U$6.VOUT2, X6-4.1
- net A: now also A.P$1, AH.S@1, AL.D@25, D8.A, D9.C, TP9.P$1; no longer U$11.P$1, U$6.S@1, U$9.D@25
- net A0/URXD1: now also JP14.7, JP15.7, JP17.7, X7-2.1; no longer U3.URXD1/NPCS2/AD6/WKUP12/PB2
- net A1/UTXD1: now also JP14.8, JP15.8, JP17.8, X7-3.1; no longer U3.UTXD1/PCK2/AD7/PB3
- net A2: now also JP14.9, JP15.9, JP17.9, SJ1.1, TP3.P$1; no longer U3.TD/PCK1/PWMH3/AD0/PA17
- net A3/PWML0: now also JP14.10, JP15.10, JP17.10; no longer U3.RK/PWML0/A15/AD2/WKUP9/PA19
- net A4: now also JP14.11, JP15.11, JP17.11, X1-4.1; no longer U3.PWMH0/AD4/PB0
- net AHO: now also R12.1; no longer R7.1
- net AHS: now also R15.1; no longer R13.1
- net ALO: now also R11.1; no longer R8.1
- net B: now also B.P$1, BH.S@1, BL.D@25, D10.A, D13.C, R14.2, TP13.P$1; no longer R13.2, U$12.P$1, U$4.S@1, U$7.D@25
- net B1/ERASE: now also JP14.5, JP15.5, JP17.5; no longer U3.PB12/PWML1/ERASE
- net B2: now also JP14.6, JP15.6, JP17.6; no longer U3.RD/PCK2/A14/AD1/PA18
- net BHO: now also TP1.P$1
- net BLO: now also TP2.P$1
- net C: now also C.P$1, CH.S@1, CL.D@25, D11.A, D12.C, R13.2, TP14.P$1; no longer R14.2, U$10.P$1, U$5.S@1, U$8.D@25
- net CHO: now also R7.1; no longer R12.1
- net CHS: now also R13.1; no longer R15.1
- net CLO: now also R8.1; no longer R11.1
- net D0/TWD0: now also JP13.16, JP16.16, JP18.16, X4-2.1; no longer U3.TWD0/NPCS3/PA3
- net D1/TWCK0: now also JP13.15, JP16.15, JP18.15, X4-1.1; no longer U3.TWCK0/TCLK0/WKUP3/PA4
- net D10: now also JP13.6, JP16.6, JP18.6, X7-1.1; no longer U3.RTS0/PWMH3/XIN32/PA7
- net D2/RX0: now also JP13.14, JP16.14, JP18.14, X2-1.1; no longer U3.RXD0/NPCS3/WKUP4/PA5
- net D3/TX0: now also JP13.13, JP16.13, JP18.13, X2-2.1; no longer U3.TXD0/PCK0/PA6
- net D4/TDI: now also JP13.12, JP16.12, JP18.12, SJ1.2, U$3.DIS; no longer U3.TWD1/PWMH2/TDI/PB4
- net D5/TDO: now also JP13.11, JP16.11, JP18.11; no longer U3.TWCK1/PWML0/WKUP13/TDO/TRACESWO/PB5
- net D6/TCK: now also JP13.10, JP16.10, JP18.10; no longer U3.TCK/SWCLK/PB7
- net D7/TMS: now also JP13.9, JP16.9, JP18.9; no longer U3.TMS/SWDIO/PB6
- net D8/PWMH1: now also JP13.8, JP16.8, JP18.8, TP6.P$1; no longer U3.PWMH1/TIOB0/A18/WKUP1/PA1
- net D9/PWMH2: now also JP13.7, JP16.7, JP18.7; no longer U3.PWMH2/SCK0/DATRG/WKUP2/PA2
- net GND: now also CIN.2, COUT.2, D2.A, JP13.1, JP13.20, JP14.1, JP14.20, JP15.1, JP15.20, JP16.1, JP16.20, JP17.1, JP17.20, JP18.1, JP18.20, R1.1, RFBB.2, TP11.P$1, TP12.P$1, TP15.P$1, TP5.P$1, U$4.2, U$5.2, X1-5.1, X2-4.1, X4-4.1, X5.GND, X7-5.1; no longer C2.1, C3.1, C32.2, C33.2, C34.2, C35.2, C36.1, C37.2, C38.1, C39.2, C40.2, C41.1, C42.1, C43.1, LED1.GND, R22.1, R6.1, U$2.GND, U$2.P$2, U$2.P$3, U$21.NEG, U3.GND@2, U3.GND@34, U3.JTAGSEL, U3.TST, X1.GND@2, X1.GND@4
- net N$11: now also BH.G@1; no longer U$5.G@1
- net N$13: now also BL.G@1; no longer U$8.G@1
- net N$14: now also AL.G@1; no longer U$9.G@1
- net N$15: now also AH.G@1; no longer U$6.G@1
- net N$7: now also CH.G@1; no longer U$4.G@1
- net N$8: now also CL.G@1; no longer U$7.G@1
- net RST: now also JP13.17, JP16.17, JP18.17; no longer U3.NRST
- net S1/PWML1: now also JP14.14, JP15.14, JP17.14, TP7.P$1; no longer U3.RF/PWML1/A16/AD3/WKUP10/PA20
- net S2/PWMH0: now also JP14.15, JP15.15, JP17.15; no longer LED1.DI, U3.PWMH0/TIOA0/A17/WKUP0/PA0
- net S3/PWML2: now also JP14.16, JP15.16, JP17.16; no longer U3.TK/TIOB1/PWML2/WKUP15/PIODCEN2/PA16
- net S5/IO3: now also JP14.18, JP15.18, JP17.18; no longer U3.NPCS0/PWMH0/WKUP7/PA11
- net UDDM: now also JP14.4, JP15.4, JP17.4, X5.D-; no longer R1.1, U$2.D-
- net UDDP: now also JP14.3, JP15.3, JP17.3, X5.D+; no longer R4.1, U$2.D+
- net UVCC: now also JP14.2, JP15.2, JP17.2, X5.VBUS; no longer F1.1, R21.2, U$2.VCC
- net VMOT: now also AH.D@25, BH.D@25, CH.D@25, CIN.1, D10.C, D11.C, D8.C, U1.VIN; no longer U$21.POS, U$4.D@25, U$5.D@25, U$6.D@25
- net VSENSE: now also AL.S@1, BL.S@1, CL.S@1, D12.A, D13.A, D9.A, TP4.P$1; no longer U$7.S@1, U$8.S@1, U$9.S@1
Other:
- note removed: "Flutter Basic: SAM3S1A Flutter Pro: SAM3S2A"
- note removed: "Main Processor"
- note removed: "Max Current Output: 500mA"
- note removed: "Max Voltage Input: 16VDC"
- note removed: "USB"
- note removed: "USB Sense"
- note removed: "VCC = 3.3V Output"
- note removed: "Voltage Input"
- note removed: "Voltage Sense"
- moved on the sheet: IC1, R1, R10, R11, R12, R14, R15, R16, R17, R18, R2, R3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

Commit message: Added BOM, Added PDFs of Schematic and PCB, Updated Project Status in Readme, added video to Readme
Parts:
- R16: value 4.7 -> DNS
- R17: value 4.7 -> 88.7K
- R18: value 4.7 -> 6.04k
- U$4: value (none) -> 10uF
Connections:
- net A5 renamed S11
- net S1/PWML1 renamed S9/PWML1
- net S2/PWMH0 renamed S8/PWMH0
- net S3/PWML2 renamed S7/PWML2
Other:
- note added: "Angle Sensor"
- moved on the sheet: U$6, U$7, X6-1, X6-2, X6-3, X6-4, X6-5
Changed lines of the file:
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@@
 <part name="GND7" library="SparkFun" deviceset="GND" device=""/>
 <part name="IC1" library="linear" deviceset="OPA333" device="D"/>
-<part name="R16" library="Taylor" deviceset="RESISTOR" device="0402" value="4.7"/>
-<part name="R17" library="Taylor" deviceset="RESISTOR" device="0402" value="4.7"/>
-<part name="R18" library="Taylor" deviceset="RESISTOR" device="0402" value="4.7"/>
+<part name="R16" library="Taylor" deviceset="RESISTOR" device="0402" value="DNS"/>
+<part name="R17" library="Taylor" deviceset="RESISTOR" device="0402" value="88.7K"/>
+<part name="R18" library="Taylor" deviceset="RESISTOR" device="0402" value="6.04k"/>
 <part name="GND8" library="SparkFun" deviceset="GND" device=""/>
 <part name="GND9" library="SparkFun" deviceset="GND" device=""/>
@@
 <part name="X4" library="con-jst-xh" deviceset="04-JST" device="-B4B-XH-A"/>
 <part name="GND14" library="SparkFun" deviceset="GND" device=""/>
-<part name="U$4" library="Taylor" deviceset="CAPACITOR" device="0805"/>
+<part name="U$4" library="Taylor" deviceset="CAPACITOR" device="0805" value="10uF"/>
 <part name="GND15" library="SparkFun" deviceset="GND" device=""/>
 <part name="U$5" library="Taylor" deviceset="CAPACITOR" device="0603-CAP" value="470pF"/>
@@
 <wire x1="175.26" y1="167.64" x2="175.26" y2="254" width="0.1524" layer="94"/>
 <text x="254" y="7.62" size="3.81" layer="95">Version 1.0</text>
+<wire x1="5.08" y1="165.1" x2="101.6" y2="165.1" width="0.1524" layer="94"/>
+<wire x1="101.6" y1="165.1" x2="101.6" y2="137.16" width="0.1524" layer="94"/>
+<wire x1="101.6" y1="137.16" x2="5.08" y2="137.16" width="0.1524" layer="94"/>
+<wire x1="5.08" y1="137.16" x2="5.08" y2="165.1" width="0.1524" layer="94"/>
+<text x="15.24" y="160.02" size="1.778" layer="94">Angle Sensor</text>
 </plain>
 <instances>
@@
 <instance part="R4" gate="G$1" x="78.74" y="104.14" rot="R90"/>
 <instance part="GND17" gate="1" x="78.74" y="81.28"/>
-<instance part="X5" gate="G$1" x="111.76" y="157.48" rot="R180"/>
-<instance part="X6" gate="-1" x="497.84" y="170.18"/>
-<instance part="X6" gate="-2" x="497.84" y="165.1"/>
-<instance part="X6" gate="-3" x="497.84" y="162.56"/>
-<instance part="X6" gate="-4" x="497.84" y="160.02"/>
-<instance part="X6" gate="-5" x="497.84" y="157.48"/>
-<instance part="U$6" gate="G$1" x="454.66" y="160.02"/>
-<instance part="U$7" gate="G$1" x="472.44" y="162.56" rot="R180"/>
+<instance part="X5" gate="G$1" x="144.78" y="167.64" rot="R180"/>
+<instance part="X6" gate="-1" x="83.82" y="157.48"/>
+<instance part="X6" gate="-2" x="83.82" y="152.4"/>
+<instance part="X6" gate="-3" x="83.82" y="149.86"/>
+<instance part="X6" gate="-4" x="83.82" y="147.32"/>
+<instance part="X6" gate="-5" x="83.82" y="144.78"/>
+<instance part="U$6" gate="G$1" x="40.64" y="147.32"/>
+<instance part="U$7" gate="G$1" x="58.42" y="149.86" rot="R180"/>
 <instance part="TP11" gate="G$1" x="35.56" y="104.14"/>
 <instance part="TP12" gate="G$1" x="43.18" y="104.14"/>
 <instance part="GND18" gate="1" x="35.56" y="96.52"/>
-<instance part="STANDOFF1" gate="G$1" x="20.32" y="172.72"/>
-<instance part="STANDOFF2" gate="G$1" x="15.24" y="172.72"/>
-<instance part="STANDOFF3" gate="G$1" x="15.24" y="167.64"/>
-<instance part="STANDOFF4" gate="G$1" x="20.32" y="167.64"/>
+<instance part="STANDOFF1" gate="G$1" x="20.32" y="73.66"/>
+<instance part="STANDOFF2" gate="G$1" x="15.24" y="73.66"/>
+<instance part="STANDOFF3" gate="G$1" x="15.24" y="68.58"/>
+<instance part="STANDOFF4" gate="G$1" x="20.32" y="68.58"/>
 <instance part="TP13" gate="G$1" x="302.26" y="106.68" rot="R270"/>
 <instance part="TP14" gate="G$1" x="266.7" y="109.22" rot="R270"/>
@@
 <segment>
 <pinref part="X5" gate="G$1" pin="GND"/>
-<wire x1="114.3" y1="157.48" x2="124.46" y2="157.48" width="0.1524" layer="91"/>
-<label x="119.38" y="157.48" size="1.778" layer="95"/>
+<wire x1="147.32" y1="167.64" x2="157.48" y2="167.64" width="0.1524" layer="91"/>
+<label x="152.4" y="167.64" size="1.778" layer="95"/>
 </segment>
 <segment>
@@
 </segment>
 </net>
-<net name="S3/PWML2" class="0">
+<net name="S7/PWML2" class="0">
 <segment>
 <pinref part="U$3" gate="G$1" pin="CLI"/>
@@
 </segment>
 </net>
-<net name="S1/PWML1" class="0">
+<net name="S9/PWML1" class="0">
 <segment>
 <pinref part="U$3" gate="G$1" pin="BLI"/>
@@
 </segment>
 </net>
-<net name="S2/PWMH0" class="0">
+<net name="S8/PWMH0" class="0">
 <segment>
 <pinref part="U$3" gate="G$1" pin="/AHI"/>
@@
 <segment>
 <pinref part="X5" gate="G$1" pin="D+"/>
-<wire x1="114.3" y1="149.86" x2="124.46" y2="149.86" width="0.1524" layer="91"/>
-<label x="119.38" y="149.86" size="1.778" layer="95"/>
+<wire x1="147.32" y1="160.02" x2="157.48" y2="160.02" width="0.1524" layer="91"/>
+<label x="152.4" y="160.02" size="1.778" layer="95"/>
 </segment>
 </net>
@@
 <segment>
 <pinref part="X5" gate="G$1" pin="D-"/>
-<wire x1="114.3" y1="152.4" x2="124.46" y2="152.4" width="0.1524" layer="91"/>
-<label x="119.38" y="152.4" size="1.778" layer="95"/>
+<wire x1="147.32" y1="162.56" x2="157.48" y2="162.56" width="0.1524" layer="91"/>
+<label x="152.4" y="162.56" size="1.778" layer="95"/>
 </segment>
 </net>
@@
 <segment>
 <pinref part="X5" gate="G$1" pin="VBUS"/>
-<wire x1="114.3" y1="154.94" x2="124.46" y2="154.94" width="0.1524" layer="91"/>
-<label x="119.38" y="154.94" size="1.778" layer="95"/>
+<wire x1="147.32" y1="165.1" x2="157.48" y2="165.1" width="0.1524" layer="91"/>
+<label x="152.4" y="165.1" size="1.778" layer="95"/>
 </segment>
 </net>
@@
 </segment>
 </net>
-<net name="A5" class="0">
+<net name="S11" class="0">
 <segment>
 <wire x1="218.44" y1="200.66" x2="203.2" y2="200.66" width="0.2032" layer="91"/>
@@
 <pinref part="U$6" gate="G$1" pin="VCC"/>
 <pinref part="X6" gate="-2" pin="1"/>
-<wire x1="467.36" y1="165.1" x2="472.44" y2="165.1" width="0.1524" layer="91"/>
-<label x="472.44" y="165.1" size="1.778" layer="95"/>
+<wire x1="53.34" y1="152.4" x2="58.42" y2="152.4" width="0.1524" layer="91"/>
+<label x="58.42" y="152.4" size="1.778" layer="95"/>
 <pinref part="U$7" gate="G$1" pin="2"/>
-<wire x1="472.44" y1="165.1" x2="492.76" y2="165.1" width="0.1524" layer="91"/>
-<junction x="472.44" y="165.1"/>
+<wire x1="58.42" y1="152.4" x2="78.74" y2="152.4" width="0.1524" layer="91"/>
+<junction x="58.42" y="152.4"/>
 <pinref part="U$6" gate="G$1" pin="TCC_EN"/>
-<wire x1="467.36" y1="160.02" x2="467.36" y2="165.1" width="0.1524" layer="91"/>
+<wire x1="53.34" y1="147.32" x2="53.34" y2="152.4" width="0.1524" layer="91"/>
 </segment>
 </net>
@@
 <pinref part="X6" gate="-5" pin="1"/>
 <pinref part="U$6" gate="G$1" pin="GND"/>
-<wire x1="492.76" y1="157.48" x2="472.44" y2="157.48" width="0.1524" layer="91"/>
+<wire x1="78.74" y1="144.78" x2="58.42" y2="144.78" width="0.1524" layer="91"/>
 <pinref part="U$7" gate="G$1" pin="1"/>
-<wire x1="472.44" y1="157.48" x2="467.36" y2="157.48" width="0.1524" layer="91"/>
-<junction x="472.44" y="157.48"/>
+<wire x1="58.42" y1="144.78" x2="53.34" y2="144.78" width="0.1524" layer="91"/>
+<junction x="58.42" y="144.78"/>
 </segment>
 </net>
@@
 <segment>
 <pinref part="U$6" gate="G$1" pin="VOUT2"/>
-<wire x1="431.8" y1="162.56" x2="421.64" y2="162.56" width="0.1524" layer="91"/>
-<label x="421.64" y="162.56" size="1.778" layer="95"/>
+<wire x1="17.78" y1="149.86" x2="7.62" y2="149.86" width="0.1524" layer="91"/>
+<label x="7.62" y="149.86" size="1.778" layer="95"/>
 </segment>
 <segment>
 <pinref part="X6" gate="-4" pin="1"/>
-<wire x1="492.76" y1="160.02" x2="474.98" y2="160.02" width="0.1524" layer="91"/>
-<label x="480.06" y="160.02" size="1.778" layer="95"/>
+<wire x1="78.74" y1="147.32" x2="60.96" y2="147.32" width="0.1524" layer="91"/>
+<label x="66.04" y="147.32" size="1.778" layer="95"/>
 </segment>
 </net>
@@
 <segment>
 <pinref part="U$6" gate="G$1" pin="VOUT1"/>
-<wire x1="431.8" y1="165.1" x2="421.64" y2="165.1" width="0.1524" layer="91"/>
-<label x="421.64" y="165.1" size="1.778" layer="95"/>
+<wire x1="17.78" y1="152.4" x2="7.62" y2="152.4" width="0.1524" layer="91"/>
+<label x="7.62" y="152.4" size="1.778" layer="95"/>
 </segment>
 <segment>
 <pinref part="X6" gate="-3" pin="1"/>
-<wire x1="492.76" y1="162.56" x2="480.06" y2="162.56" width="0.1524" layer="91"/>
-<wire x1="480.06" y1="162.56" x2="474.98" y2="162.56" width="0.1524" layer="91"/>
-<label x="480.06" y="162.56" size="1.778" layer="95"/>
-</segment>
-</net>
+<wire x1="78.74" y1="149.86" x2="60.96" y2="149.86" width="0.1524" layer="91"/>
+<label x="66.04" y="149.86" size="1.778" layer="95"/>
+</segment>
+</net>

Commit message: Updated readme. Also pushing latest changes to board. Can't actually remember what they are.
Connections:
- net D11 renamed S0/UVCC
- net S0/CK renamed S10/CK
- net S11 renamed S11/A5
- net S4/IO2 renamed S6/IO2
- net S6/IO0 renamed S4/IO0
- net S7/B renamed S3/B
- net S8/G renamed S2/G
- net S9/R renamed S1/R
Changed lines of the file:
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@@
 </segment>
 </net>
-<net name="S6/IO0" class="0">
+<net name="S4/IO0" class="0">
 <segment>
 <wire x1="198.12" y1="182.88" x2="200.66" y2="182.88" width="0.2032" layer="91"/>
@@
 </segment>
 </net>
-<net name="S4/IO2" class="0">
+<net name="S6/IO2" class="0">
 <segment>
 <wire x1="198.12" y1="187.96" x2="200.66" y2="187.96" width="0.2032" layer="91"/>
@@
 </segment>
 </net>
-<net name="S0/CK" class="0">
+<net name="S10/CK" class="0">
 <segment>
 <wire x1="218.44" y1="198.12" x2="203.2" y2="198.12" width="0.1524" layer="91"/>
@@
 </segment>
 </net>
-<net name="S7/B" class="0">
+<net name="S3/B" class="0">
 <segment>
 <wire x1="248.92" y1="182.88" x2="251.46" y2="182.88" width="0.1524" layer="91"/>
@@
 </segment>
 </net>
-<net name="S9/R" class="0">
+<net name="S1/R" class="0">
 <segment>
 <wire x1="248.92" y1="187.96" x2="251.46" y2="187.96" width="0.1524" layer="91"/>
@@
 </segment>
 </net>
-<net name="D11" class="0">
+<net name="S0/UVCC" class="0">
 <segment>
 <wire x1="248.92" y1="190.5" x2="251.46" y2="190.5" width="0.2032" layer="91"/>
@@
 </segment>
 </net>
-<net name="S11" class="0">
-<segment>
-<wire x1="218.44" y1="200.66" x2="203.2" y2="200.66" width="0.2032" layer="91"/>
-<label x="208.28" y="200.66" size="1.778" layer="95"/>
-<pinref part="JP14" gate="G$1" pin="12"/>
-<pinref part="JP15" gate="G$1" pin="12"/>
-<wire x1="203.2" y1="200.66" x2="200.66" y2="200.66" width="0.2032" layer="91"/>
-<wire x1="200.66" y1="200.66" x2="198.12" y2="200.66" width="0.2032" layer="91"/>
-<junction x="200.66" y="200.66"/>
-<pinref part="JP17" gate="G$1" pin="12"/>
-<junction x="203.2" y="200.66"/>
-</segment>
-<segment>
-<pinref part="X1" gate="-3" pin="1"/>
-<wire x1="292.1" y1="213.36" x2="276.86" y2="213.36" width="0.1524" layer="91"/>
-<label x="279.4" y="213.36" size="1.778" layer="95"/>
-</segment>
-</net>
 <net name="A4" class="0">
 <segment>
@@
 </segment>
 </net>
-<net name="S8/G" class="0">
+<net name="S2/G" class="0">
 <segment>
 <wire x1="248.92" y1="185.42" x2="251.46" y2="185.42" width="0.1524" layer="91"/>
@@
 </segment>
 </net>
+<net name="S11/A5" class="0">
+<segment>
+<wire x1="218.44" y1="200.66" x2="203.2" y2="200.66" width="0.2032" layer="91"/>
+<label x="208.28" y="200.66" size="1.778" layer="95"/>
+<pinref part="JP14" gate="G$1" pin="12"/>
+<pinref part="JP15" gate="G$1" pin="12"/>
+<wire x1="203.2" y1="200.66" x2="200.66" y2="200.66" width="0.2032" layer="91"/>
+<wire x1="200.66" y1="200.66" x2="198.12" y2="200.66" width="0.2032" layer="91"/>
+<junction x="200.66" y="200.66"/>
+<pinref part="JP17" gate="G$1" pin="12"/>
+<junction x="203.2" y="200.66"/>
+</segment>
+<segment>
+<pinref part="X1" gate="-3" pin="1"/>
+<wire x1="292.1" y1="213.36" x2="276.86" y2="213.36" width="0.1524" layer="91"/>
+<label x="279.4" y="213.36" size="1.778" layer="95"/>
+</segment>
+</net>

Commit message: Updated wiring for better compatibility with Flutter, fixed current sense filter, removed angle sensor.
Parts:
- removed U$6: KMZ60_MAG_ANGLE_SENSOR, Taylor:KMZ60_MAG_ANGLE_SENSOR
- removed U$7: 0.22uF, Taylor:CAPACITOR0805
- removed X6: 05-JST-B5B-XH-A, con-jst-xh:05-JST-B5B-XH-A
- added D14: (no value), SparkFun-DiscreteSemi:DIODESOD123
- added R5: 6.04k, Taylor:RESISTOR0402
- added R6: 6.04k, SparkFun-Capacitors:CAP0805
Connections:
- removed net GND2: U$6.GND, U$7.1, X6-5.1
- removed net S8/PWMH0: JP14.15, JP15.15, JP17.15, U$3./AHI
- removed net S9/PWML1: JP14.14, JP15.14, JP17.14, TP7.P$1, U$3.BLI
- removed net VCC2: U$6.TCC_EN, U$6.VCC, U$7.2, X6-2.1
- removed net VOUT1: U$6.VOUT1, X6-3.1
- removed net VOUT2: U$6.VOUT2, X6-4.1
- new net N$3: IC1.+IN, R5.2, R6.1
- new net RAW: D14.C, JP13.19, JP16.19, JP18.19, X1-1.1
- net +12V: now also D14.A; no longer JP13.19, JP16.19, JP18.19, X1-1.1
- net D5/TDO: now also TP7.P$1, U$3.BLI
- net GND: now also R6.2
- net S2/G: now also U$3./AHI
- net VSENSE: now also R5.1; no longer IC1.+IN
Other:
- note removed: "Angle Sensor"
- moved on the sheet: IC1, JP13, JP16, R16, R17, R18, TP3, TP4

Commit message: Added angle sensor. Checked in latest board version.
Parts:
- added IC2: 7805TV, linear:7805TV
- added J1: (no value), SparkFun-Connectors:M01PTH
- added J2: (no value), SparkFun-Connectors:M02PTH
- added R19, R20, R21: 20k, Taylor:RESISTOR0402
- added R22, R23: (no value), Taylor:RESISTOR0603
- added U$1: MOSFETSOT23, Taylor:MOSFETSOT23
- R5: value 6.04k -> 1k; device Taylor:RESISTOR0402 -> Taylor:RESISTOR0603
- R6: value 6.04k -> 0.1uF
Connections:
- new net N$10: J2.2, U$1.D@25
- new net N$4: IC2.VO, J1.1
- new net N$5: JP14.14, JP15.14, JP17.14
- new net N$6: JP14.15, JP15.15, JP17.15
- net +12V: now also IC2.VI, J2.1
- net A0/URXD1: now also R20.2, R22.2, R23.1
- net A1/UTXD1: now also R21.2
- net D10: now also R19.2
- net D7/TMS: now also U$1.G@1
- net GND: now also IC2.GND, R23.2, U$1.S@1
- net VCC: now also R19.1, R20.1, R21.1, R22.1
Other:
- moved on the sheet: +, -, A, AH, AL, B, BH, BL, C, C1, C4, CH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
